File: GameConsole.kicad_sch (KiCad schematic)
At the start: 22 parts, among them J1 Display, J2 SD, J3 PCM5100, J4 Conn_01x02, SW1 SW_Push, SW2 SW_Push, SW3 SW_Push, SW4 SW_Push, SW5 SW_Push, SW6 SW_Push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

Commit message: v1
Other:
- company: (none) -> JensFZ
- title: (none) -> Game Console
Changed lines of the file:
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@@
 	(generator_version "8.0")
 	(paper "A4")
+	(title_block
+		(title "Game Console")
+		(date "2024-06-06")
+		(rev "Rev. 1")
+		(company "JensFZ")
+	)
 	(junction
 		(at 217.17 88.9)
@@
 		)
 		(instances
-			(project "BBC"
+			(project "GameConsole"
 				(path "/f390af48-df43-4320-b418-9f5882e857f8"
 					(reference "#PWR027")
@@
 		)
 		(instances
-			(project "BBC"
+			(project "GameConsole"
 				(path "/f390af48-df43-4320-b418-9f5882e857f8"
 					(reference "#PWR05")
@@
 		)
 		(instances
-			(project "BBC"
+			(project "GameConsole"
 				(path "/f390af48-df43-4320-b418-9f5882e857f8"
 					(reference "J4")
@@
 		)
 		(instances
-			(project "BBC"
+			(project "GameConsole"
 				(path "/f390af48-df43-4320-b418-9f5882e857f8"
 					(reference "#PWR025")
@@
 		)
 		(instances
-			(project "BBC"
+			(project "GameConsole"
 				(path "/f390af48-df43-4320-b418-9f5882e857f8"
 					(reference "#PWR02")
@@
 		)
 		(instances
-			(project "BBC"
+			(project "GameConsole"
 				(path "/f390af48-df43-4320-b418-9f5882e857f8"
 					(reference "#PWR06")
@@
 		)
 		(instances
-			(project "BBC"
+			(project "GameConsole"
 				(path "/f390af48-df43-4320-b418-9f5882e857f8"
 					(reference "J2")
@@
 		)
 		(instances
-			(project "BBC"
+			(project "GameConsole"
 				(path "/f390af48-df43-4320-b418-9f5882e857f8"
 					(reference "#PWR017")
@@
 		)
 		(instances
-			(project "BBC"
+			(project "GameConsole"
 				(path "/f390af48-df43-4320-b418-9f5882e857f8"
 					(reference "SW2")
@@
 		)
 		(instances
-			(project "BBC"
+			(project "GameConsole"
 				(path "/f390af48-df43-4320-b418-9f5882e857f8"
 					(reference "#PWR07")
@@
 		)
 		(instances
-			(project "BBC"
+			(project "GameConsole"
 				(path "/f390af48-df43-4320-b418-9f5882e857f8"
 					(reference "#PWR022")
@@
 		)
 		(instances
-			(project "BBC"
+			(project "GameConsole"
 				(path "/f390af48-df43-4320-b418-9f5882e857f8"
 					(reference "R1")
@@
 		)
 		(instances
-			(project "BBC"
+			(project "GameConsole"
 				(path "/f390af48-df43-4320-b418-9f5882e857f8"
 					(reference "#PWR010")
@@
 		)
 		(instances
-			(project "BBC"
+			(project "GameConsole"
 				(path "/f390af48-df43-4320-b418-9f5882e857f8"
 					(reference "#PWR014")
@@
 		)
 		(instances
-			(project "BBC"
+			(project "GameConsole"
 				(path "/f390af48-df43-4320-b418-9f5882e857f8"
 					(reference "#PWR04")
@@
 		)
 		(instances
-			(project "BBC"
+			(project "GameConsole"
 				(path "/f390af48-df43-4320-b418-9f5882e857f8"
 					(reference "J3")
@@
 		)
 		(instances
-			(project "BBC"
+			(project "GameConsole"
 				(path "/f390af48-df43-4320-b418-9f5882e857f8"
 					(reference "#PWR020")
@@
 		)
 		(instances
-			(project "BBC"
+			(project "GameConsole"
 				(path "/f390af48-df43-4320-b418-9f5882e857f8"
 					(reference "#PWR019")
@@
 		)
 		(instances
-			(project "BBC"
+			(project "GameConsole"
 				(path "/f390af48-df43-4320-b418-9f5882e857f8"
 					(reference "#PWR021")
@@
 		)
 		(instances
-			(project "BBC"
+			(project "GameConsole"
 				(path "/f390af48-df43-4320-b418-9f5882e857f8"
 					(reference "#PWR012")
@@
 		)
 		(instances
-			(project "BBC"
+			(project "GameConsole"
 				(path "/f390af48-df43-4320-b418-9f5882e857f8"
 					(reference "R4")
@@
 		)
 		(instances
-			(project "BBC"
+			(project "GameConsole"
 				(path "/f390af48-df43-4320-b418-9f5882e857f8"
 					(reference "#PWR015")
@@
 		)
 		(instances
-			(project "BBC"
+			(project "GameConsole"
 				(path "/f390af48-df43-4320-b418-9f5882e857f8"
 					(reference "#PWR013")
@@
 		)
 		(instances
-			(project "BBC"
+			(project "GameConsole"
 				(path "/f390af48-df43-4320-b418-9f5882e857f8"
 					(reference "SW6")
@@
 		)
 		(instances
-			(project "BBC"
+			(project "GameConsole"
 				(path "/f390af48-df43-4320-b418-9f5882e857f8"
 					(reference "SW3")
@@
 		)
 		(instances
-			(project "BBC"
+			(project "GameConsole"
 				(path "/f390af48-df43-4320-b418-9f5882e857f8"
 					(reference "R2")
@@
 		)
 		(instances
-			(project "BBC"
+			(project "GameConsole"
 				(path "/f390af48-df43-4320-b418-9f5882e857f8"
 					(reference "#PWR01")
@@
 		)
 		(instances
-			(project "BBC"
+			(project "GameConsole"
 				(path "/f390af48-df43-4320-b418-9f5882e857f8"
 					(reference "R5")
@@
 		)
 		(instances
-			(project "BBC"
+			(project "GameConsole"
 				(path "/f390af48-df43-4320-b418-9f5882e857f8"
 					(reference "SW1")
@@
 		)
 		(instances
-			(project "BBC"
+			(project "GameConsole"
 				(path "/f390af48-df43-4320-b418-9f5882e857f8"
 					(reference "#PWR034")
@@
 		)
 		(instances
-			(project "BBC"
+			(project "GameConsole"
 				(path "/f390af48-df43-4320-b418-9f5882e857f8"
 					(reference "#PWR026")
@@
 		)
 		(instances
-			(project "BBC"
+			(project "GameConsole"
 				(path "/f390af48-df43-4320-b418-9f5882e857f8"
 					(reference "#PWR08")
@@
 		)
 		(instances
-			(project "BBC"
+			(project "GameConsole"
 				(path "/f390af48-df43-4320-b418-9f5882e857f8"
 					(reference "U4")
@@
 		)
 		(instances
-			(project "BBC"
+			(project "GameConsole"
 				(path "/f390af48-df43-4320-b418-9f5882e857f8"
 					(reference "D1")
@@
 		)
 		(instances
-			(project "BBC"
+			(project "GameConsole"
 				(path "/f390af48-df43-4320-b418-9f5882e857f8"
 					(reference "#PWR03")
@@
 		)
 		(instances
-			(project "BBC"
+			(project "GameConsole"
 				(path "/f390af48-df43-4320-b418-9f5882e857f8"
 					(reference "#PWR033")
@@
 		)
 		(instances
-			(project "BBC"
+			(project "GameConsole"
 				(path "/f390af48-df43-4320-b418-9f5882e857f8"
 					(reference "SW7")
@@
 		)
 		(instances
-			(project "BBC"
+			(project "GameConsole"
 				(path "/f390af48-df43-4320-b418-9f5882e857f8"
 					(reference "#PWR016")
@@
 		)
 		(instances
-			(project "BBC"
+			(project "GameConsole"
 				(path "/f390af48-df43-4320-b418-9f5882e857f8"
 					(reference "#PWR023")
@@
 		)
 		(instances
-			(project "BBC"
+			(project "GameConsole"
 				(path "/f390af48-df43-4320-b418-9f5882e857f8"
 					(reference "#PWR011")
@@
 		)
 		(instances
-			(project "BBC"
+			(project "GameConsole"
 				(path "/f390af48-df43-4320-b418-9f5882e857f8"
 					(reference "R8")
@@
 		)
 		(instances
-			(project "BBC"
+			(project "GameConsole"
 				(path "/f390af48-df43-4320-b418-9f5882e857f8"
 					(reference "SW4")
@@
 		)
 		(instances
-			(project "BBC"
+			(project "GameConsole"
 				(path "/f390af48-df43-4320-b418-9f5882e857f8"
 					(reference "#PWR018")
@@
 		)
 		(instances
-			(project "BBC"
+			(project "GameConsole"
 				(path "/f390af48-df43-4320-b418-9f5882e857f8"
 					(reference "#PWR024")
@@
 		)
 		(instances
-			(project "BBC"
+			(project "GameConsole"
 				(path "/f390af48-df43-4320-b418-9f5882e857f8"
 					(reference "R7")
@@
 		)
 		(instances
-			(project "BBC"
+			(project "GameConsole"
 				(path "/f390af48-df43-4320-b418-9f5882e857f8"
 					(reference "SW8")
@@
 		)
 		(instances
-			(project "BBC"
+			(project "GameConsole"
 				(path "/f390af48-df43-4320-b418-9f5882e857f8"
 					(reference "R6")
@@
 		)
 		(instances
-			(project "BBC"
+			(project "GameConsole"
 				(path "/f390af48-df43-4320-b418-9f5882e857f8"
 					(reference "J1")
@@
 		)
 		(instances
-			(project "BBC"
+			(project "GameConsole"
 				(path "/f390af48-df43-4320-b418-9f5882e857f8"
 					(reference "#PWR09")
@@
 		)
 		(instances
-			(project "BBC"
+			(project "GameConsole"
 				(path "/f390af48-df43-4320-b418-9f5882e857f8"
 					(reference "SW5")
@@
 		)
 		(instances
-			(project "BBC"
+			(project "GameConsole"
 				(path "/f390af48-df43-4320-b418-9f5882e857f8"
 					(reference "R3")

Commit message: Pinheader durch Socket ersetzt
Parts:
- J1: footprint Connector_PinHeader_2.54mm:PinHeader_1x08_P2.54mm_Vertical -> Connector_PinSocket_2.54mm:PinSocket_1x08_P2.54mm_Vertical
- J2, J3: footprint Connector_PinHeader_2.54mm:PinHeader_1x06_P2.54mm_Vertical -> Connector_PinSocket_2.54mm:PinSocket_1x06_P2.54mm_Vertical
Changed lines of the file:
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@@
 			)
 		)
-		(property "Footprint" "Connector_PinHeader_2.54mm:PinHeader_1x06_P2.54mm_Vertical"
+		(property "Footprint" "Connector_PinSocket_2.54mm:PinSocket_1x06_P2.54mm_Vertical"
 			(at 240.03 27.94 0)
 			(effects
@@
 			)
 		)
-		(property "Footprint" "Connector_PinHeader_2.54mm:PinHeader_1x06_P2.54mm_Vertical"
+		(property "Footprint" "Connector_PinSocket_2.54mm:PinSocket_1x06_P2.54mm_Vertical"
 			(at 266.7 29.21 0)
 			(effects
@@
 			)
 		)
-		(property "Footprint" "Connector_PinHeader_2.54mm:PinHeader_1x08_P2.54mm_Vertical"
+		(property "Footprint" "Connector_PinSocket_2.54mm:PinSocket_1x08_P2.54mm_Vertical"
 			(at 209.55 29.21 0)
 			(effects
